Commit message: robot code

File: body.urdf (robot description, URDF)
Before this commit: robot robot, 3 links, 2 joints
Links:
- removed link BackLeg
Joints:
- removed joint Torso_BackLeg

Commit message: sensors

File: body.urdf (robot description, URDF)
Before this commit: robot robot, 2 links, 1 joints
Links:
- added link BackLeg, mass 1; collision box size=1 1 1; visual box size=1 1 1
Joints:
- added joint Torso_BackLeg: type revolute, parent Torso, child BackLeg, origin xyz=-0.5 0 1 rpy=0 0 0, axis 0 1 0, limit lower=-3.14159 upper=3.14159 effort=0.0 velocity=0.0
- joint Torso_FrontLeg: origin xyz=2.5 0 1 rpy=0 0 0 -> xyz=0.5 0 1 rpy=0 0 0

Commit message: completed bipedal

File: body.urdf (robot description, URDF)
Before this commit: robot robot, 9 links, 8 joints
Links:
- removed link BackLeg
- removed link BackLowerLeg
- removed link FrontLeg
- removed link FrontLowerLeg
- removed link LeftLeg
- removed link LeftLowerLeg
- removed link RightLeg
- removed link RightLowerLeg
- added link Hip, mass 1; collision box size=0.5 1 0.2; visual box size=0.5 1 0.2
- added link LeftFemur, mass 1; collision box size=0.2 0.2 1; visual box size=0.2 0.2 1
- added link LeftFoot, mass 1; collision box size=0.4 0.4 0.2; visual box size=0.4 0.4 0.2
- added link LeftTibia, mass 1; collision box size=0.2 0.2 0.8; visual box size=0.2 0.2 0.8
- added link RightFemur, mass 1; collision box size=0.2 0.2 1; visual box size=0.2 0.2 1
- added link RightFoot, mass 1; collision box size=0.4 0.4 0.2; visual box size=0.4 0.4 0.2
- added link RightTibia, mass 1; collision box size=0.2 0.2 0.8; visual box size=0.2 0.2 0.8
- link Torso: geometry collision box size=0.5 0.5 1; visual box size=0.5 0.5 1
Joints:
- removed joint BackLeg_BackLowerLeg
- removed joint FrontLeg_FrontLowerLeg
- removed joint LeftLeg_LeftLowerLeg
- removed joint RightLeg_RightLowerLeg
- removed joint Torso_BackLeg
- removed joint Torso_FrontLeg
- removed joint Torso_LeftLeg
- removed joint Torso_RightLeg
- added joint Hip_LeftFemur: type revolute, parent Hip, child LeftFemur, origin xyz=0 -0.5 0 rpy=0 0 0, axis 0 1 0, limit lower=-3.14159 upper=3.14159 effort=0.0 velocity=0.0
- added joint Hip_RightFemur: type revolute, parent Hip, child RightFemur, origin xyz=0 0.5 0 rpy=0 0 0, axis 0 1 0 , limit lower=-3.14159 upper=3.14159 effort=0.0 velocity=0.0
- added joint LeftFemur_LeftTibia: type revolute, parent LeftFemur, child LeftTibia, origin xyz=0 0 -1 rpy=0 0 0, axis 0 1 0, limit lower=-3.14159 upper=3.14159 effort=0.0 velocity=0.0
- added joint LeftTibia_LeftFoot: type revolute, parent LeftTibia, child LeftFoot, origin xyz=0 0 -0.4 rpy=0 0 0, axis 0 1 0, limit lower=-3.14159 upper=3.14159 effort=0.0 velocity=0.0
- added joint RightFemur_RightTibia: type revolute, parent RightFemur, child RightTibia, origin xyz=0 0 -1 rpy=0 0 0, axis 0 1 0, limit lower=-3.14159 upper=3.14159 effort=0.0 velocity=0.0
- added joint RightTibia_RightFoot: type revolute, parent RightTibia, child RightFoot, origin xyz=0 0 -0.4 rpy=0 0 0, axis 0 1 0, limit lower=-3.14159 upper=3.14159 effort=0.0 velocity=0.0
- added joint Torso_Hip: type revolute, parent Torso, child Hip, origin xyz=0 0 1.5 rpy=0 0 0, axis 0 0 1, limit lower=-3.14159 upper=3.14159 effort=0.0 velocity=0.0

Commit message: finished robot, starting stairs

File: body.urdf (robot description, URDF)
Before this commit: robot robot, 8 links, 7 joints
Links:
- link LeftFemur: geometry collision box size=0.2 0.2 0.8; visual box size=0.2 0.2 0.8
- link LeftTibia: geometry collision box size=0.2 0.2 0.6; visual box size=0.2 0.2 0.6
- link RightFemur: geometry collision box size=0.2 0.2 0.8; visual box size=0.2 0.2 0.8
- link RightTibia: geometry collision box size=0.2 0.2 0.6; visual box size=0.2 0.2 0.6
Joints:
- joint LeftFemur_LeftTibia: origin xyz=0 0 -1 rpy=0 0 0 -> xyz=0 0 -0.8 rpy=0 0 0
- joint LeftTibia_LeftFoot: origin xyz=0 0 -0.4 rpy=0 0 0 -> xyz=0 0 -0.6 rpy=0 0 0
- joint RightFemur_RightTibia: origin xyz=0 0 -1 rpy=0 0 0 -> xyz=0 0 -0.8 rpy=0 0 0
- joint RightTibia_RightFoot: origin xyz=0 0 -0.4 rpy=0 0 0 -> xyz=0 0 -0.6 rpy=0 0 0

Commit message: finished bipedal got it to somewhat work

File: body.urdf (robot description, URDF)
Before this commit: robot robot, 8 links, 7 joints
Links:
- link Torso: geometry collision box size=0.25 0.25 0.5; visual box size=0.25 0.25 0.5
Joints:
- joint Torso_Hip: origin xyz=0 0 1.5 rpy=0 0 0 -> xyz=0 0 2.5 rpy=0 0 0

Commit message: random length + size

File: body.urdf (robot description, URDF)
Before this commit: robot robot, 8 links, 7 joints
Links:
- removed link Hip
- removed link LeftFemur
- removed link LeftFoot
- removed link LeftTibia
- removed link RightFemur
- removed link RightFoot
- removed link RightTibia
- removed link Torso
- added link Body0, mass 1; collision box size=0.5525900571815241 0.30927390038169167 0.33168115664034553; visual box size=0.5525900571815241 0.30927390038169167 0.33168115664034553
- added link Body1, mass 1; collision box size=0.5743759779158146 0.32608808040499354 0.15036153471926972; visual box size=0.5743759779158146 0.32608808040499354 0.15036153471926972
- added link Body2, mass 1; collision box size=0.6177877137870486 0.20442433154553352 0.1287536712470693; visual box size=0.6177877137870486 0.20442433154553352 0.1287536712470693
- added link Body3, mass 1; collision box size=0.8628596484197576 0.36499285763062084 0.21712860505090978; visual box size=0.8628596484197576 0.36499285763062084 0.21712860505090978
- added link Body4, mass 1; collision box size=0.5129381641030415 0.37912834645500837 0.48320544805278387; visual box size=0.5129381641030415 0.37912834645500837 0.48320544805278387
- added link Body5, mass 1; collision box size=0.6583271303598613 0.1972618264855433 0.32500038227850214; visual box size=0.6583271303598613 0.1972618264855433 0.32500038227850214
- added link Body6, mass 1; collision box size=0.9800205092861554 0.23880298089455707 0.3517251085453612; visual box size=0.9800205092861554 0.23880298089455707 0.3517251085453612
Joints:
- removed joint Hip_LeftFemur
- removed joint Hip_RightFemur
- removed joint LeftFemur_LeftTibia
- removed joint LeftTibia_LeftFoot
- removed joint RightFemur_RightTibia
- removed joint RightTibia_RightFoot
- removed joint Torso_Hip
- added joint Body0_Body1: type revolute, parent Body0, child Body1, origin xyz=0.27629502859076205 0 0.16584057832017277 rpy=0 0 0, axis 0 0 1, limit lower=-3.14159 upper=3.14159 effort=0.0 velocity=0.0
- added joint Body1_Body2: type revolute, parent Body1, child Body2, origin xyz=0.2871879889579073 0 0 rpy=0 0 0, axis 0 0 1, limit lower=-3.14159 upper=3.14159 effort=0.0 velocity=0.0
- added joint Body2_Body3: type revolute, parent Body2, child Body3, origin xyz=0.3088938568935243 0 0 rpy=0 0 0, axis 0 0 1, limit lower=-3.14159 upper=3.14159 effort=0.0 velocity=0.0
- added joint Body3_Body4: type revolute, parent Body3, child Body4, origin xyz=0.4314298242098788 0 0 rpy=0 0 0, axis 0 0 1, limit lower=-3.14159 upper=3.14159 effort=0.0 velocity=0.0
- added joint Body4_Body5: type revolute, parent Body4, child Body5, origin xyz=0.25646908205152075 0 0 rpy=0 0 0, axis 0 0 1, limit lower=-3.14159 upper=3.14159 effort=0.0 velocity=0.0
- added joint Body5_Body6: type revolute, parent Body5, child Body6, origin xyz=0.3291635651799307 0 0 rpy=0 0 0, axis 0 0 1, limit lower=-3.14159 upper=3.14159 effort=0.0 velocity=0.0

Commit message: finished snake

File: body.urdf (robot description, URDF)
Before this commit: robot robot, 7 links, 6 joints
Links:
- removed link Body2
- removed link Body3
- removed link Body4
- removed link Body5
- removed link Body6
- link Body0: geometry collision box size=0.6129474314155764 0.3187289057395491 0.16159215185759002; visual box size=0.6129474314155764 0.3187289057395491 0.16159215185759002
- link Body1: geometry collision box size=0.3924054483894499 0.21962645178269136 0.34557431748193645; visual box size=0.3924054483894499 0.21962645178269136 0.34557431748193645
Joints:
- removed joint Body1_Body2
- removed joint Body2_Body3
- removed joint Body3_Body4
- removed joint Body4_Body5
- removed joint Body5_Body6
- joint Body0_Body1: origin xyz=0.27629502859076205 0 0.16584057832017277 rpy=0 0 0 -> xyz=0.3064737157077882 0 0.08079607592879501 rpy=0 0 0

Commit message: updated weights

File: body.urdf (robot description, URDF)
Before this commit: robot robot, 2 links, 1 joints
Links:
- added link Body10, mass 1; collision box size=0.6522641055542155 0.40775309044276176 0.26163350620117043; visual box size=0.6522641055542155 0.40775309044276176 0.26163350620117043
- added link Body2, mass 1; collision box size=0.8163251541215588 0.20579050476251515 0.3276074166629248; visual box size=0.8163251541215588 0.20579050476251515 0.3276074166629248
- added link Body3, mass 1; collision box size=0.2934723306746321 0.34607977259224443 0.46245585886543816; visual box size=0.2934723306746321 0.34607977259224443 0.46245585886543816
- added link Body4, mass 1; collision box size=0.9592149519597409 0.3965186682816578 0.4987918234196761; visual box size=0.9592149519597409 0.3965186682816578 0.4987918234196761
- added link Body5, mass 1; collision box size=0.1118214334096298 0.14331626757339677 0.488256148822093; visual box size=0.1118214334096298 0.14331626757339677 0.488256148822093
- added link Body6, mass 1; collision box size=0.48958918343479063 0.15549514577817353 0.41429427627395043; visual box size=0.48958918343479063 0.15549514577817353 0.41429427627395043
- added link Body7, mass 1; collision box size=0.5314372746039532 0.48811285905679547 0.31778483165295157; visual box size=0.5314372746039532 0.48811285905679547 0.31778483165295157
- added link Body8, mass 1; collision box size=0.780519175951639 0.2007053861599733 0.15771221895064308; visual box size=0.780519175951639 0.2007053861599733 0.15771221895064308
- added link Body9, mass 1; collision box size=0.6455130061743692 0.3144480504963476 0.4332510507750774; visual box size=0.6455130061743692 0.3144480504963476 0.4332510507750774
- link Body0: geometry collision box size=0.6592669112032228 0.21608717719202974 0.26615962626076584; visual box size=0.6592669112032228 0.21608717719202974 0.26615962626076584
- link Body1: geometry collision box size=0.12249358469639708 0.24777468462801588 0.23135833386792004; visual box size=0.12249358469639708 0.24777468462801588 0.23135833386792004
Joints:
- added joint Body1_Body2: type revolute, parent Body1, child Body2, origin xyz=0.12249358469639708 0 0 rpy=0 0 0, axis 0 0 1, limit lower=-3.14159 upper=3.14159 effort=0.0 velocity=0.0
- added joint Body2_Body3: type revolute, parent Body2, child Body3, origin xyz=0.8163251541215588 0 0 rpy=0 0 0, axis 0 0 1, limit lower=-3.14159 upper=3.14159 effort=0.0 velocity=0.0
- added joint Body3_Body4: type revolute, parent Body3, child Body4, origin xyz=0.2934723306746321 0 0 rpy=0 0 0, axis 0 0 1, limit lower=-3.14159 upper=3.14159 effort=0.0 velocity=0.0
- added joint Body4_Body5: type revolute, parent Body4, child Body5, origin xyz=0.9592149519597409 0 0 rpy=0 0 0, axis 0 0 1, limit lower=-3.14159 upper=3.14159 effort=0.0 velocity=0.0
- added joint Body5_Body6: type revolute, parent Body5, child Body6, origin xyz=0.1118214334096298 0 0 rpy=0 0 0, axis 0 0 1, limit lower=-3.14159 upper=3.14159 effort=0.0 velocity=0.0
- added joint Body6_Body7: type revolute, parent Body6, child Body7, origin xyz=0.48958918343479063 0 0 rpy=0 0 0, axis 0 0 1, limit lower=-3.14159 upper=3.14159 effort=0.0 velocity=0.0
- added joint Body7_Body8: type revolute, parent Body7, child Body8, origin xyz=0.5314372746039532 0 0 rpy=0 0 0, axis 0 0 1, limit lower=-3.14159 upper=3.14159 effort=0.0 velocity=0.0
- added joint Body8_Body9: type revolute, parent Body8, child Body9, origin xyz=0.780519175951639 0 0 rpy=0 0 0, axis 0 0 1, limit lower=-3.14159 upper=3.14159 effort=0.0 velocity=0.0
- added joint Body9_Body10: type revolute, parent Body9, child Body10, origin xyz=0.6455130061743692 0 0 rpy=0 0 0, axis 0 0 1, limit lower=-3.14159 upper=3.14159 effort=0.0 velocity=0.0
- joint Body0_Body1: origin xyz=0.3064737157077882 0 0.08079607592879501 rpy=0 0 0 -> xyz=0.3296334556016114 0 0.13307981313038292 rpy=0 0 0

Commit message: added a bunch of random things and OOPd

File: body.urdf (robot description, URDF)
Before this commit: robot robot, 11 links, 10 joints
Links:
- removed link Body10
- removed link Body8
- removed link Body9
- link Body0: geometry collision box size=0.5832816933457781 0.8995547033589129 0.6130787832222389; visual box size=0.5832816933457781 0.8995547033589129 0.6130787832222389
- link Body1: geometry collision box size=0.7062911254274185 0.15666675362512125 0.8463862324895707; visual box size=0.7062911254274185 0.15666675362512125 0.8463862324895707
- link Body2: geometry collision box size=0.5690927514291295 0.6173009998365012 0.2103804890135338; visual box size=0.5690927514291295 0.6173009998365012 0.2103804890135338
- link Body3: geometry collision box size=0.7459257506764139 0.9984662842337185 0.1822441725810225; visual box size=0.7459257506764139 0.9984662842337185 0.1822441725810225
- link Body4: geometry collision box size=0.22926449243191838 0.8563022050091909 0.9135715958523211; visual box size=0.22926449243191838 0.8563022050091909 0.9135715958523211
- link Body5: geometry collision box size=0.35417183155637366 0.8124639635173087 0.8827781089674276; visual box size=0.35417183155637366 0.8124639635173087 0.8827781089674276
- link Body6: geometry collision box size=0.5812791394661748 0.842157341910121 0.553087177678866; visual box size=0.5812791394661748 0.842157341910121 0.553087177678866
- link Body7: geometry collision box size=0.2585074654195845 0.7731318326426369 0.4692621110669062; visual box size=0.2585074654195845 0.7731318326426369 0.4692621110669062
Joints:
- removed joint Body7_Body8
- removed joint Body8_Body9
- removed joint Body9_Body10
- joint Body0_Body1: axis 0 0 1 -> 0 1 0; origin xyz=0.3296334556016114 0 0.13307981313038292 rpy=0 0 0 -> xyz=0.29164084667288903 0 0.3065393916111194 rpy=0 0 0
- joint Body1_Body2: axis 0 0 1 -> 1 0 0; origin xyz=0.12249358469639708 0 0 rpy=0 0 0 -> xyz=0.7062911254274185 0 0 rpy=0 0 0
- joint Body2_Body3: origin xyz=0.8163251541215588 0 0 rpy=0 0 0 -> xyz=0.5690927514291295 0 0 rpy=0 0 0
- joint Body3_Body4: axis 0 0 1 -> 0 1 0; origin xyz=0.2934723306746321 0 0 rpy=0 0 0 -> xyz=0.7459257506764139 0 0 rpy=0 0 0
- joint Body4_Body5: axis 0 0 1 -> 1 0 0; origin xyz=0.9592149519597409 0 0 rpy=0 0 0 -> xyz=0.22926449243191838 0 0 rpy=0 0 0
- joint Body5_Body6: axis 0 0 1 -> 1 0 0; origin xyz=0.1118214334096298 0 0 rpy=0 0 0 -> xyz=0.35417183155637366 0 0 rpy=0 0 0
- joint Body6_Body7: axis 0 0 1 -> 1 0 0; origin xyz=0.48958918343479063 0 0 rpy=0 0 0 -> xyz=0.5812791394661748 0 0 rpy=0 0 0

Commit message: added one sided legs

File: body.urdf (robot description, URDF)
Before this commit: robot robot, 8 links, 7 joints
Links:
- added link Body10, mass 1; collision box size=0.12813925035292278 1 1; visual box size=0.12813925035292278 1 1
- added link Body8, mass 1; collision box size=0.464766925140119 1 1; visual box size=0.464766925140119 1 1
- added link Body9, mass 1; collision box size=0.03713918123730829 1 1; visual box size=0.03713918123730829 1 1
- link Body0: geometry collision box size=0.5815019038863494 0.4632127200704488 0.15541080565560683; visual box size=0.5815019038863494 0.4632127200704488 0.15541080565560683
- link Body1: geometry collision box size=0.25422747413985136 0.16894933052487773 0.9522492123969759; visual box size=0.25422747413985136 0.16894933052487773 0.9522492123969759
- link Body2: geometry collision box size=0.9667669930442931 0.2645269438916297 0.24501338138191453; visual box size=0.9667669930442931 0.2645269438916297 0.24501338138191453
- link Body3: geometry collision box size=0.3350182455137754 0.8654220414697316 0.799017720083343; visual box size=0.3350182455137754 0.8654220414697316 0.799017720083343
- link Body4: geometry collision box size=0.48304614350720865 0.8023775434165081 0.531978458557414; visual box size=0.48304614350720865 0.8023775434165081 0.531978458557414
- link Body5: geometry collision box size=0.6467394888834682 0.3801798293369476 0.605066179544785; visual box size=0.6467394888834682 0.3801798293369476 0.605066179544785
- link Body6: geometry collision box size=0.3012958850130568 0.1844488337257855 0.8581681653119982; visual box size=0.3012958850130568 0.1844488337257855 0.8581681653119982
- link Body7: geometry collision box size=0.004598452417190062 1 1; visual box size=0.004598452417190062 1 1
Joints:
- removed joint Body6_Body7
- added joint Body0_Body7: type revolute, parent Body0, child Body7, origin xyz=0.2907509519431747 0.2316063600352244 0 rpy=0 0 0, axis 0 0 1, limit lower=-3.14159 upper=3.14159 effort=0.0 velocity=0.0
- added joint Body0_Body8: type revolute, parent Body0, child Body8, origin xyz=0.2907509519431747 -0.2316063600352244 0 rpy=0 0 0, axis 0 0 1, limit lower=-3.14159 upper=3.14159 effort=0.0 velocity=0.0
- added joint Body6_Body10: type revolute, parent Body6, child Body10, origin xyz=0.1506479425065284 -0.09222441686289275 0 rpy=0 0 0, axis 0 0 1, limit lower=-3.14159 upper=3.14159 effort=0.0 velocity=0.0
- added joint Body6_Body9: type revolute, parent Body6, child Body9, origin xyz=0.1506479425065284 0.09222441686289275 0 rpy=0 0 0, axis 0 0 1, limit lower=-3.14159 upper=3.14159 effort=0.0 velocity=0.0
- joint Body0_Body1: axis 0 1 0 -> 0 0 1; origin xyz=0.29164084667288903 0 0.3065393916111194 rpy=0 0 0 -> xyz=0.2907509519431747 0 0.07770540282780342 rpy=0 0 0
- joint Body1_Body2: origin xyz=0.7062911254274185 0 0 rpy=0 0 0 -> xyz=0.25422747413985136 0 0 rpy=0 0 0
- joint Body2_Body3: origin xyz=0.5690927514291295 0 0 rpy=0 0 0 -> xyz=0.9667669930442931 0 0 rpy=0 0 0
- joint Body3_Body4: axis 0 1 0 -> 0 0 1; origin xyz=0.7459257506764139 0 0 rpy=0 0 0 -> xyz=0.3350182455137754 0 0 rpy=0 0 0
- joint Body4_Body5: origin xyz=0.22926449243191838 0 0 rpy=0 0 0 -> xyz=0.48304614350720865 0 0 rpy=0 0 0
- joint Body5_Body6: axis 1 0 0 -> 0 1 0; origin xyz=0.35417183155637366 0 0 rpy=0 0 0 -> xyz=0.6467394888834682 0 0 rpy=0 0 0

Commit message: added rpy for joint rotation

File: body.urdf (robot description, URDF)
Before this commit: robot robot, 11 links, 10 joints
Links:
- added link Body11, mass 1; collision box size=0.09576484228647221 1 1; visual box size=0.09576484228647221 1 1
- added link Body12, mass 1; collision box size=0.7155173111670798 1 1; visual box size=0.7155173111670798 1 1
- added link Body13, mass 1; collision box size=0.5269199235367491 1 1; visual box size=0.5269199235367491 1 1
- added link Body14, mass 1; collision box size=0.6132535141889723 1 1; visual box size=0.6132535141889723 1 1
- link Body0: geometry collision box size=0.2569632156167317 0.485340096278044 0.1544918289411423; visual box size=0.2569632156167317 0.485340096278044 0.1544918289411423
- link Body1: geometry collision box size=0.6019145706721999 0.22186645711654174 0.6929686631572294; visual box size=0.6019145706721999 0.22186645711654174 0.6929686631572294
- link Body10: geometry collision box size=0.5582399478604619 0.4565124570428457 0.8852425723345384; visual box size=0.5582399478604619 0.4565124570428457 0.8852425723345384
- link Body2: geometry collision box size=0.15583106383138315 0.321793005074287 0.4715335554172574; visual box size=0.15583106383138315 0.321793005074287 0.4715335554172574
- link Body3: geometry collision box size=0.9388602874161053 0.5984282206933873 0.3694517632248008; visual box size=0.9388602874161053 0.5984282206933873 0.3694517632248008
- link Body4: geometry collision box size=0.24602627797995757 0.11066061875969407 0.5758743065206086; visual box size=0.24602627797995757 0.11066061875969407 0.5758743065206086
- link Body5: geometry collision box size=0.6255370456430065 0.9466681426240926 0.7684128718841056; visual box size=0.6255370456430065 0.9466681426240926 0.7684128718841056
- link Body6: geometry collision box size=0.6483055897082395 0.9480969323528747 0.11009210039014627; visual box size=0.6483055897082395 0.9480969323528747 0.11009210039014627
- link Body7: geometry collision box size=0.5620135000939767 0.32493769700047703 0.47553641471899677; visual box size=0.5620135000939767 0.32493769700047703 0.47553641471899677
- link Body8: geometry collision box size=0.18375744587293863 0.8504519743510845 0.7826833115455125; visual box size=0.18375744587293863 0.8504519743510845 0.7826833115455125
- link Body9: geometry collision box size=0.7748803507765833 0.5217743907269363 0.13084526848382952; visual box size=0.7748803507765833 0.5217743907269363 0.13084526848382952
Joints:
- removed joint Body0_Body7
- removed joint Body0_Body8
- removed joint Body6_Body10
- removed joint Body6_Body9
- added joint Body3_Body11: type revolute, parent Body3, child Body11, origin xyz=0.46943014370805264 0.29921411034669365 0 rpy=0 1 0, axis 0 0 1, limit lower=-3.14159 upper=3.14159 effort=0.0 velocity=0.0
- added joint Body3_Body12: type revolute, parent Body3, child Body12, origin xyz=0.46943014370805264 -0.29921411034669365 0 rpy=0 1 0, axis 0 0 1, limit lower=-3.14159 upper=3.14159 effort=0.0 velocity=0.0
- added joint Body5_Body13: type revolute, parent Body5, child Body13, origin xyz=0.31276852282150325 0.4733340713120463 0 rpy=0 1 0, axis 1 0 0, limit lower=-3.14159 upper=3.14159 effort=0.0 velocity=0.0
- added joint Body5_Body14: type revolute, parent Body5, child Body14, origin xyz=0.31276852282150325 -0.4733340713120463 0 rpy=0 1 0, axis 1 0 0, limit lower=-3.14159 upper=3.14159 effort=0.0 velocity=0.0
- added joint Body6_Body7: type revolute, parent Body6, child Body7, origin xyz=0.6483055897082395 0 0 rpy=0 0 0, axis 1 0 0, limit lower=-3.14159 upper=3.14159 effort=0.0 velocity=0.0
- added joint Body7_Body8: type revolute, parent Body7, child Body8, origin xyz=0.5620135000939767 0 0 rpy=0 0 0, axis 0 1 0, limit lower=-3.14159 upper=3.14159 effort=0.0 velocity=0.0
- added joint Body8_Body9: type revolute, parent Body8, child Body9, origin xyz=0.18375744587293863 0 0 rpy=0 0 0, axis 0 0 1, limit lower=-3.14159 upper=3.14159 effort=0.0 velocity=0.0
- added joint Body9_Body10: type revolute, parent Body9, child Body10, origin xyz=0.7748803507765833 0 0 rpy=0 0 0, axis 0 0 1, limit lower=-3.14159 upper=3.14159 effort=0.0 velocity=0.0
- joint Body0_Body1: origin xyz=0.2907509519431747 0 0.07770540282780342 rpy=0 0 0 -> xyz=0.12848160780836584 0 0.07724591447057115 rpy=0 0 0
- joint Body1_Body2: origin xyz=0.25422747413985136 0 0 rpy=0 0 0 -> xyz=0.6019145706721999 0 0 rpy=0 0 0
- joint Body2_Body3: origin xyz=0.9667669930442931 0 0 rpy=0 0 0 -> xyz=0.15583106383138315 0 0 rpy=0 0 0
- joint Body3_Body4: origin xyz=0.3350182455137754 0 0 rpy=0 0 0 -> xyz=0.9388602874161053 0 0 rpy=0 0 0
- joint Body4_Body5: axis 1 0 0 -> 0 0 1; origin xyz=0.48304614350720865 0 0 rpy=0 0 0 -> xyz=0.24602627797995757 0 0 rpy=0 0 0
- joint Body5_Body6: axis 0 1 0 -> 1 0 0; origin xyz=0.6467394888834682 0 0 rpy=0 0 0 -> xyz=0.6255370456430065 0 0 rpy=0 0 0
