Commit message: added rpy for joint rotation

File: body.urdf (robot description, URDF)
Before this commit: robot robot, 15 links, 14 joints
Links:
- added link Body15, mass 1; collision box size=0.25418996978628683 1 1; visual box size=0.25418996978628683 1 1
- added link Body16, mass 1; collision box size=0.23943871828579963 1 1; visual box size=0.23943871828579963 1 1
- added link Body17, mass 1; collision box size=0.4046357343990976 1 1; visual box size=0.4046357343990976 1 1
- added link Body18, mass 1; collision box size=0.0979745161777105 0.19545518480777124 0.17731835524571316; visual box size=0.0979745161777105 0.19545518480777124 0.17731835524571316
- added link Body19, mass 1; collision box size=0.06307492682852782 1 1; visual box size=0.06307492682852782 1 1
- added link Body20, mass 1; collision box size=0.20083761836629366 1 1; visual box size=0.20083761836629366 1 1
- added link Body21, mass 1; collision box size=0.11569651432326744 1 1; visual box size=0.11569651432326744 1 1
- link Body0: geometry collision box size=0.9198791234062605 0.655403377027737 0.7960748108197541; visual box size=0.9198791234062605 0.655403377027737 0.7960748108197541
- link Body1: geometry collision box size=0.6858812830086249 0.38506730287630975 0.3522791740429192; visual box size=0.6858812830086249 0.38506730287630975 0.3522791740429192
- link Body10: geometry collision box size=0.6357113289401858 1.3888202788221062 0.9895199231190874; visual box size=0.6357113289401858 1.3888202788221062 0.9895199231190874
- link Body11: geometry collision box size=0.6651818919783469 1 1; visual box size=0.6651818919783469 1 1
- link Body12: geometry collision box size=0.3949036290535103 1 1; visual box size=0.3949036290535103 1 1
- link Body13: geometry collision box size=0.4041681093921405 1 1; visual box size=0.4041681093921405 1 1
- link Body14: geometry collision box size=0.5260832341873471 0.3316006443499302 1.390326812365715; visual box size=0.5260832341873471 0.3316006443499302 1.390326812365715
- link Body2: geometry collision box size=0.7092647699011363 0.8637156369718083 0.9469659581777351; visual box size=0.7092647699011363 0.8637156369718083 0.9469659581777351
- link Body3: geometry collision box size=0.6079828131058327 0.1530442392205032 0.11297803615282682; visual box size=0.6079828131058327 0.1530442392205032 0.11297803615282682
- link Body4: geometry collision box size=0.31099464010614747 0.837621176577614 0.5687384077987683; visual box size=0.31099464010614747 0.837621176577614 0.5687384077987683
- link Body5: geometry collision box size=0.2466480414564084 0.7054647323581876 0.2958507053016991; visual box size=0.2466480414564084 0.7054647323581876 0.2958507053016991
- link Body6: geometry collision box size=0.3102980381335712 0.2964793649068196 0.5271596447757567; visual box size=0.3102980381335712 0.2964793649068196 0.5271596447757567
- link Body7: geometry collision box size=0.11323522073152646 1 1; visual box size=0.11323522073152646 1 1
- link Body8: geometry collision box size=0.4990201754683954 1 1; visual box size=0.4990201754683954 1 1
- link Body9: geometry collision box size=0.31504966163867104 1 1; visual box size=0.31504966163867104 1 1
Joints:
- removed joint Body3_Body11
- removed joint Body3_Body12
- removed joint Body5_Body13
- removed joint Body5_Body14
- removed joint Body5_Body6
- removed joint Body7_Body8
- removed joint Body9_Body10
- added joint Body10_Body11: type revolute, parent Body10, child Body11, origin xyz=0 1.3888202788221062 -0.4947599615595437 rpy=0 0 0, axis 0 1 0, limit lower=-3.14159 upper=3.14159 effort=0.0 velocity=0.0
- added joint Body12_Body13: type revolute, parent Body12, child Body13, origin xyz=0 -1 -0.5 rpy=0 0 0, axis 0 1 0, limit lower=-3.14159 upper=3.14159 effort=0.0 velocity=0.0
- added joint Body14_Body15: type revolute, parent Body14, child Body15, origin xyz=0 0.3316006443499302 -0.6951634061828575 rpy=0 0 0, axis 0 1 0, limit lower=-3.14159 upper=3.14159 effort=0.0 velocity=0.0
- added joint Body16_Body17: type revolute, parent Body16, child Body17, origin xyz=0 -1 -0.5 rpy=0 0 0, axis 0 1 0, limit lower=-3.14159 upper=3.14159 effort=0.0 velocity=0.0
- added joint Body18_Body19: type revolute, parent Body18, child Body19, origin xyz=0 0.19545518480777124 -0.08865917762285658 rpy=0 0 0, axis 1 0 0, limit lower=-3.14159 upper=3.14159 effort=0.0 velocity=0.0
- added joint Body1_Body6: type revolute, parent Body1, child Body6, origin xyz=0.34294064150431247 0.19253365143815487 0 rpy=0 0 0, axis 1 0 0, limit lower=-3.14159 upper=3.14159 effort=0.0 velocity=0.0
- added joint Body1_Body8: type revolute, parent Body1, child Body8, origin xyz=0.34294064150431247 -0.19253365143815487 0 rpy=0 0 0, axis 1 0 0, limit lower=-3.14159 upper=3.14159 effort=0.0 velocity=0.0
- added joint Body20_Body21: type revolute, parent Body20, child Body21, origin xyz=0 -1 -0.5 rpy=0 0 0, axis 1 0 0, limit lower=-3.14159 upper=3.14159 effort=0.0 velocity=0.0
- added joint Body2_Body10: type revolute, parent Body2, child Body10, origin xyz=0.35463238495056815 0.43185781848590415 0 rpy=0 0 0, axis 0 1 0, limit lower=-3.14159 upper=3.14159 effort=0.0 velocity=0.0
- added joint Body2_Body12: type revolute, parent Body2, child Body12, origin xyz=0.35463238495056815 -0.43185781848590415 0 rpy=0 0 0, axis 0 1 0, limit lower=-3.14159 upper=3.14159 effort=0.0 velocity=0.0
- added joint Body3_Body14: type revolute, parent Body3, child Body14, origin xyz=0.30399140655291634 0.0765221196102516 0 rpy=0 0 0, axis 0 1 0, limit lower=-3.14159 upper=3.14159 effort=0.0 velocity=0.0
- added joint Body3_Body16: type revolute, parent Body3, child Body16, origin xyz=0.30399140655291634 -0.0765221196102516 0 rpy=0 0 0, axis 0 1 0, limit lower=-3.14159 upper=3.14159 effort=0.0 velocity=0.0
- added joint Body4_Body18: type revolute, parent Body4, child Body18, origin xyz=0.15549732005307373 0.418810588288807 0 rpy=0 0 0, axis 1 0 0, limit lower=-3.14159 upper=3.14159 effort=0.0 velocity=0.0
- added joint Body4_Body20: type revolute, parent Body4, child Body20, origin xyz=0.15549732005307373 -0.418810588288807 0 rpy=0 0 0, axis 1 0 0, limit lower=-3.14159 upper=3.14159 effort=0.0 velocity=0.0
- joint Body0_Body1: axis 0 0 1 -> 1 0 0; origin xyz=0.12848160780836584 0 0.07724591447057115 rpy=0 0 0 -> xyz=0.4599395617031303 0 2.398037405409877 rpy=0 0 0
- joint Body1_Body2: origin xyz=0.6019145706721999 0 0 rpy=0 0 0 -> xyz=0.6858812830086249 0 0 rpy=0 0 0
- joint Body2_Body3: axis 0 0 1 -> 0 1 0; origin xyz=0.15583106383138315 0 0 rpy=0 0 0 -> xyz=0.7092647699011363 0 0 rpy=0 0 0
- joint Body3_Body4: axis 0 0 1 -> 0 1 0; origin xyz=0.9388602874161053 0 0 rpy=0 0 0 -> xyz=0.6079828131058327 0 0 rpy=0 0 0
- joint Body4_Body5: axis 0 0 1 -> 1 0 0; origin xyz=0.24602627797995757 0 0 rpy=0 0 0 -> xyz=0.31099464010614747 0 0 rpy=0 0 0
- joint Body6_Body7: origin xyz=0.6483055897082395 0 0 rpy=0 0 0 -> xyz=0 0.2964793649068196 -0.26357982238787836 rpy=0 0 0
- joint Body8_Body9: axis 0 0 1 -> 1 0 0; origin xyz=0.18375744587293863 0 0 rpy=0 0 0 -> xyz=0 -1 -0.5 rpy=0 0 0

Commit message: created leg class

File: body.urdf (robot description, URDF)
Before this commit: robot robot, 22 links, 21 joints
Links:
- removed link Body10
- removed link Body11
- removed link Body12
- removed link Body13
- removed link Body14
- removed link Body15
- removed link Body16
- removed link Body17
- removed link Body18
- removed link Body19
- removed link Body20
- removed link Body21
- removed link Body8
- removed link Body9
- link Body0: geometry collision box size=0.11340963925611836 0.83093449190615 0.6970568915050342; visual box size=0.11340963925611836 0.83093449190615 0.6970568915050342
- link Body1: geometry collision box size=0.9749003212776971 0.43028252312353577 0.5721506278104266; visual box size=0.9749003212776971 0.43028252312353577 0.5721506278104266
- link Body2: geometry collision box size=0.12332577416556109 0.838828389637362 0.6251764667596383; visual box size=0.12332577416556109 0.838828389637362 0.6251764667596383
- link Body3: geometry collision box size=0.8402378187983789 0.07716276659483341 0.13318581750175926; visual box size=0.8402378187983789 0.07716276659483341 0.13318581750175926
- link Body4: geometry collision box size=0.48301627444291495 1 1; visual box size=0.48301627444291495 1 1
- link Body5: geometry collision box size=0.05172264586242172 0.18473610782736785 0.5585847054177573; visual box size=0.05172264586242172 0.18473610782736785 0.5585847054177573
- link Body6: geometry collision box size=0.075576194067038 1 1; visual box size=0.075576194067038 1 1
- link Body7: geometry collision box size=0.08134761896983914 1 1; visual box size=0.08134761896983914 1 1
Joints:
- removed joint Body10_Body11
- removed joint Body12_Body13
- removed joint Body14_Body15
- removed joint Body16_Body17
- removed joint Body18_Body19
- removed joint Body1_Body6
- removed joint Body1_Body8
- removed joint Body20_Body21
- removed joint Body2_Body10
- removed joint Body2_Body12
- removed joint Body2_Body3
- removed joint Body3_Body14
- removed joint Body3_Body16
- removed joint Body4_Body18
- removed joint Body4_Body20
- removed joint Body4_Body5
- removed joint Body6_Body7
- removed joint Body8_Body9
- added joint Body1_Body3: type revolute, parent Body1, child Body3, origin xyz=0.48745016063884855 0.21514126156176788 0 rpy=0 0 0, axis 0 0 1, limit lower=-3.14159 upper=3.14159 effort=0.0 velocity=0.0
- added joint Body2_Body5: type revolute, parent Body2, child Body5, origin xyz=0.061662887082780546 0.419414194818681 0 rpy=0 0 0, axis 0 1 0, limit lower=-3.14159 upper=3.14159 effort=0.0 velocity=0.0
- added joint Body2_Body7: type revolute, parent Body2, child Body7, origin xyz=0.061662887082780546 -0.419414194818681 0 rpy=0 0 0, axis 0 0 1, limit lower=-3.14159 upper=3.14159 effort=0.0 velocity=0.0
- added joint Body5_Body6: type revolute, parent Body5, child Body6, origin xyz=0 0.18473610782736785 -0.27929235270887864 rpy=0 0 0, axis 0 0 1, limit lower=-3.14159 upper=3.14159 effort=0.0 velocity=0.0
- joint Body0_Body1: axis 1 0 0 -> 0 1 0; origin xyz=0.4599395617031303 0 2.398037405409877 rpy=0 0 0 -> xyz=0.05670481962805918 0 2.348528445752517 rpy=0 0 0
- joint Body1_Body2: axis 1 0 0 -> 0 0 1; origin xyz=0.6858812830086249 0 0 rpy=0 0 0 -> xyz=0.9749003212776971 0 0 rpy=0 0 0
- joint Body3_Body4: axis 0 1 0 -> 0 0 1; origin xyz=0.6079828131058327 0 0 rpy=0 0 0 -> xyz=0 0.07716276659483341 -0.06659290875087963 rpy=0 0 0

Commit message: fixed parent child bug

File: body.urdf (robot description, URDF)
Before this commit: robot robot, 8 links, 7 joints
Links:
- added link Body10, mass 1; collision box size=0.011957982325688534 0.9275444579900919 0.03386360915022243; visual box size=0.011957982325688534 0.9275444579900919 0.03386360915022243
- added link Body11, mass 1; collision box size=0.002488984346281363 0.6754162975504118 0.053488432278668833; visual box size=0.002488984346281363 0.6754162975504118 0.053488432278668833
- added link Body12, mass 1; collision box size=0.14508554054624137 0.5862782035020958 0.3701907583590312; visual box size=0.14508554054624137 0.5862782035020958 0.3701907583590312
- added link Body13, mass 1; collision box size=0.13633034912494502 0.12016061362533119 0.6486607855782643; visual box size=0.13633034912494502 0.12016061362533119 0.6486607855782643
- added link Body14, mass 1; collision box size=0.07083642306080279 0.4261663683423915 0.30808729505449767; visual box size=0.07083642306080279 0.4261663683423915 0.30808729505449767
- added link Body15, mass 1; collision box size=0.045658408079501986 0.21779058119008757 0.0534576656922585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; visual box size=0.045658408079501986 0.21779058119008757 0.0534576656922585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
- added link Body16, mass 1; collision box size=0.03653907851998913 0.3161178899898788 0.0661386552327193; visual box size=0.03653907851998913 0.3161178899898788 0.0661386552327193
- added link Body17, mass 1; collision box size=0.01734816686145601 0.20450571422063799 0.00294040685148190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; visual box size=0.01734816686145601 0.20450571422063799 0.00294040685148190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
- added link Body18, mass 1; collision box size=0.10701953790210217 0.12752009579756216 0.1481504428397885; visual box size=0.10701953790210217 0.12752009579756216 0.1481504428397885
- added link Body19, mass 1; collision box size=0.08736076451775202 0.02339626904089281 0.016028846261757594; visual box size=0.08736076451775202 0.02339626904089281 0.016028846261757594
- added link Body20, mass 1; collision box size=0.05449728863563515 0.4562217858639856 0.021563364707709816; visual box size=0.05449728863563515 0.4562217858639856 0.021563364707709816
- added link Body21, mass 1; collision box size=0.024392894261554353 0.416225399437 0.016175328347614634; visual box size=0.024392894261554353 0.416225399437 0.016175328347614634
- added link Body22, mass 1; collision box size=0.3372736739104485 0.7059128774781921 0.31734542185323916; visual box size=0.3372736739104485 0.7059128774781921 0.31734542185323916
- added link Body23, mass 1; collision box size=0.2907729607424911 0.43762489268483823 0.26284386030363727; visual box size=0.2907729607424911 0.43762489268483823 0.26284386030363727
- added link Body24, mass 1; collision box size=0.1894667852174788 0.13139828939910972 0.1789388512576581; visual box size=0.1894667852174788 0.13139828939910972 0.1789388512576581
- added link Body25, mass 1; collision box size=0.05007546098782768 0.018263407868506984 0.02433101502202737; visual box size=0.05007546098782768 0.018263407868506984 0.02433101502202737
- added link Body8, mass 1; collision box size=0.5542063732753455 0.34580592637214963 0.08594768398871724; visual box size=0.5542063732753455 0.34580592637214963 0.08594768398871724
- added link Body9, mass 1; collision box size=0.260131659519378 0.04872308693249624 0.15555098666972492; visual box size=0.260131659519378 0.04872308693249624 0.15555098666972492
- link Body0: geometry collision box size=0.9377961095255218 0.4361562708087684 0.4613884614650836; visual box size=0.9377961095255218 0.4361562708087684 0.4613884614650836
- link Body1: geometry collision box size=0.7179331956033698 0.5464497255668367 0.1210188522204735; visual box size=0.7179331956033698 0.5464497255668367 0.1210188522204735
- link Body2: geometry collision box size=0.15873846218031484 0.9449917762284894 0.7062306613696726; visual box size=0.15873846218031484 0.9449917762284894 0.7062306613696726
- link Body3: geometry collision box size=0.19011154817370146 0.7115529613114251 0.31520852656519927; visual box size=0.19011154817370146 0.7115529613114251 0.31520852656519927
- link Body4: geometry collision box size=0.11299601147428873 0.7038073100975022 0.39518670128215894; visual box size=0.11299601147428873 0.7038073100975022 0.39518670128215894
- link Body5: geometry collision box size=0.40333913305330704 0.8179775890156016 0.5445720600054794; visual box size=0.40333913305330704 0.8179775890156016 0.5445720600054794
- link Body6: geometry collision box size=0.6217003252505 0.224182805599199 0.026813303628514154; visual box size=0.6217003252505 0.224182805599199 0.026813303628514154
- link Body7: geometry collision box size=0.3659562275891558 0.20497135660593882 0.014126890960007818; visual box size=0.3659562275891558 0.20497135660593882 0.014126890960007818
Joints:
- removed joint Body1_Body3
- removed joint Body2_Body5
- removed joint Body2_Body7
- removed joint Body5_Body6
- added joint Body10_Body11: type revolute, parent Body10, child Body11, origin xyz=0 0.9275444579900919 -0.016931804575111214 rpy=0 0 0, axis 1 0 0, limit lower=-3.14159 upper=3.14159 effort=0.0 velocity=0.0
- added joint Body12_Body13: type revolute, parent Body12, child Body13, origin xyz=0 -0.5862782035020958 -0.1850953791795156 rpy=0 0 0, axis 0 0 1, limit lower=-3.14159 upper=3.14159 effort=0.0 velocity=0.0
- added joint Body14_Body15: type revolute, parent Body14, child Body15, origin xyz=0 0.4261663683423915 -0.15404364752724883 rpy=0 0 0, axis 1 0 0, limit lower=-3.14159 upper=3.14159 effort=0.0 velocity=0.0
- added joint Body16_Body17: type revolute, parent Body16, child Body17, origin xyz=0 -0.3161178899898788 -0.03306932761635965 rpy=0 0 0, axis 0 1 0, limit lower=-3.14159 upper=3.14159 effort=0.0 velocity=0.0
- added joint Body18_Body19: type revolute, parent Body18, child Body19, origin xyz=0 0.12752009579756216 -0.07407522141989425 rpy=0 0 0, axis 1 0 0, limit lower=-3.14159 upper=3.14159 effort=0.0 velocity=0.0
- added joint Body1_Body6: type revolute, parent Body1, child Body6, origin xyz=0.3589665978016849 0.27322486278341834 0 rpy=0 0 0, axis 0 1 0, limit lower=-3.14159 upper=3.14159 effort=0.0 velocity=0.0
- added joint Body1_Body8: type revolute, parent Body1, child Body8, origin xyz=0.3589665978016849 -0.27322486278341834 0 rpy=0 0 0, axis 0 0 1, limit lower=-3.14159 upper=3.14159 effort=0.0 velocity=0.0
- added joint Body20_Body21: type revolute, parent Body20, child Body21, origin xyz=0 -0.4562217858639856 -0.010781682353854908 rpy=0 0 0, axis 1 0 0, limit lower=-3.14159 upper=3.14159 effort=0.0 velocity=0.0
- added joint Body22_Body23: type revolute, parent Body22, child Body23, origin xyz=0 0.7059128774781921 -0.15867271092661958 rpy=0 0 0, axis 1 0 0, limit lower=-3.14159 upper=3.14159 effort=0.0 velocity=0.0
- added joint Body24_Body25: type revolute, parent Body24, child Body25, origin xyz=0 -0.13139828939910972 -0.08946942562882905 rpy=0 0 0, axis 0 1 0, limit lower=-3.14159 upper=3.14159 effort=0.0 velocity=0.0
- added joint Body2_Body10: type revolute, parent Body2, child Body10, origin xyz=0.07936923109015742 0.4724958881142447 0 rpy=0 0 0, axis 1 0 0, limit lower=-3.14159 upper=3.14159 effort=0.0 velocity=0.0
- added joint Body2_Body12: type revolute, parent Body2, child Body12, origin xyz=0.07936923109015742 -0.4724958881142447 0 rpy=0 0 0, axis 0 1 0, limit lower=-3.14159 upper=3.14159 effort=0.0 velocity=0.0
- added joint Body2_Body3: type revolute, parent Body2, child Body3, origin xyz=0.15873846218031484 0 0 rpy=0 0 0, axis 1 0 0, limit lower=-3.14159 upper=3.14159 effort=0.0 velocity=0.0
- added joint Body3_Body14: type revolute, parent Body3, child Body14, origin xyz=0.09505577408685073 0.35577648065571255 0 rpy=0 0 0, axis 1 0 0, limit lower=-3.14159 upper=3.14159 effort=0.0 velocity=0.0
- added joint Body3_Body16: type revolute, parent Body3, child Body16, origin xyz=0.09505577408685073 -0.35577648065571255 0 rpy=0 0 0, axis 0 1 0, limit lower=-3.14159 upper=3.14159 effort=0.0 velocity=0.0
- added joint Body4_Body18: type revolute, parent Body4, child Body18, origin xyz=0.05649800573714436 0.3519036550487511 0 rpy=0 0 0, axis 0 0 1, limit lower=-3.14159 upper=3.14159 effort=0.0 velocity=0.0
- added joint Body4_Body20: type revolute, parent Body4, child Body20, origin xyz=0.05649800573714436 -0.3519036550487511 0 rpy=0 0 0, axis 1 0 0, limit lower=-3.14159 upper=3.14159 effort=0.0 velocity=0.0
- added joint Body4_Body5: type revolute, parent Body4, child Body5, origin xyz=0.11299601147428873 0 0 rpy=0 0 0, axis 1 0 0, limit lower=-3.14159 upper=3.14159 effort=0.0 velocity=0.0
- added joint Body5_Body22: type revolute, parent Body5, child Body22, origin xyz=0.20166956652665352 0.4089887945078008 0 rpy=0 0 0, axis 0 1 0, limit lower=-3.14159 upper=3.14159 effort=0.0 velocity=0.0
- added joint Body5_Body24: type revolute, parent Body5, child Body24, origin xyz=0.20166956652665352 -0.4089887945078008 0 rpy=0 0 0, axis 0 0 1, limit lower=-3.14159 upper=3.14159 effort=0.0 velocity=0.0
- added joint Body6_Body7: type revolute, parent Body6, child Body7, origin xyz=0 0.224182805599199 -0.013406651814257077 rpy=0 0 0, axis 0 0 1, limit lower=-3.14159 upper=3.14159 effort=0.0 velocity=0.0
- added joint Body8_Body9: type revolute, parent Body8, child Body9, origin xyz=0 -0.34580592637214963 -0.04297384199435862 rpy=0 0 0, axis 0 1 0, limit lower=-3.14159 upper=3.14159 effort=0.0 velocity=0.0
- joint Body0_Body1: axis 0 1 0 -> 0 0 1; origin xyz=0.05670481962805918 0 2.348528445752517 rpy=0 0 0 -> xyz=0.4688980547627609 0 2.2306942307325417 rpy=0 0 0
- joint Body1_Body2: origin xyz=0.9749003212776971 0 0 rpy=0 0 0 -> xyz=0.7179331956033698 0 0 rpy=0 0 0
- joint Body3_Body4: axis 0 0 1 -> 1 0 0; origin xyz=0 0.07716276659483341 -0.06659290875087963 rpy=0 0 0 -> xyz=0.19011154817370146 0 0 rpy=0 0 0
