Commit message: finished - will have to add weight dimensinos

File: body.urdf (robot description, URDF)
Before this commit: robot robot, 26 links, 25 joints
Links:
- removed link Body16
- removed link Body17
- removed link Body18
- removed link Body19
- removed link Body20
- removed link Body21
- removed link Body22
- removed link Body23
- removed link Body24
- removed link Body25
- link Body0: geometry collision box size=0.18121430008089162 0.25293276718959634 0.20573749923399293; visual box size=0.18121430008089162 0.25293276718959634 0.20573749923399293
- link Body1: geometry collision box size=0.7776446127363325 0.606200143378221 0.4080987302800033; visual box size=0.7776446127363325 0.606200143378221 0.4080987302800033
- link Body10: geometry collision box size=0.31159088346945124 0.3393051675011771 0.18106684929408545; visual box size=0.31159088346945124 0.3393051675011771 0.18106684929408545
- link Body11: geometry collision box size=0.04464432025214566 0.1888029052717333 0.15765654531011894; visual box size=0.04464432025214566 0.1888029052717333 0.15765654531011894
- link Body12: geometry collision box size=0.499317470116161 0.09174995987187068 0.7374041458070142; visual box size=0.499317470116161 0.09174995987187068 0.7374041458070142
- link Body13: geometry collision box size=0.11946353435964328 0.011422718404856244 0.979354928793334; visual box size=0.11946353435964328 0.011422718404856244 0.979354928793334
- link Body14: geometry collision box size=0.6617783610816057 0.11039933576914382 0.42780472215457327; visual box size=0.6617783610816057 0.11039933576914382 0.42780472215457327
- link Body15: geometry collision box size=0.6128630366054518 0.10294326609692601 0.5319630404705021; visual box size=0.6128630366054518 0.10294326609692601 0.5319630404705021
- link Body2: geometry collision box size=0.629994333130818 0.5364391938059476 0.8972400841692829; visual box size=0.629994333130818 0.5364391938059476 0.8972400841692829
- link Body3: geometry collision box size=0.8855042618485532 0.12706424263053331 0.6518921865651908; visual box size=0.8855042618485532 0.12706424263053331 0.6518921865651908
- link Body4: geometry collision box size=0.2618435257102146 0.34961574996824235 0.6477605000516001; visual box size=0.2618435257102146 0.34961574996824235 0.6477605000516001
- link Body5: geometry collision box size=0.13317971826030514 0.3969393948555852 0.21272201407332958; visual box size=0.13317971826030514 0.3969393948555852 0.21272201407332958
- link Body6: geometry collision box size=0.5445898099373764 0.6285472885228587 0.19377304839519027; visual box size=0.5445898099373764 0.6285472885228587 0.19377304839519027
- link Body7: geometry collision box size=0.09794696916001029 0.6448962579812038 0.004526074336097626; visual box size=0.09794696916001029 0.6448962579812038 0.004526074336097626
- link Body8: geometry collision box size=0.2561819212353715 0.7678398653959259 0.8738020632665383; visual box size=0.2561819212353715 0.7678398653959259 0.8738020632665383
- link Body9: geometry collision box size=0.24231208549957287 0.6337330670946001 0.6430757372613612; visual box size=0.24231208549957287 0.6337330670946001 0.6430757372613612
Joints:
- removed joint Body16_Body17
- removed joint Body18_Body19
- removed joint Body1_Body8
- removed joint Body20_Body21
- removed joint Body22_Body23
- removed joint Body24_Body25
- removed joint Body2_Body12
- removed joint Body3_Body16
- removed joint Body3_Body4
- removed joint Body4_Body18
- removed joint Body4_Body20
- removed joint Body5_Body22
- removed joint Body5_Body24
- added joint Body1_Body4: type revolute, parent Body1, child Body4, origin xyz=0.3888223063681662 0.3031000716891105 0 rpy=0 0 0, axis 1 0 0, limit lower=-3.14159 upper=3.14159 effort=0.0 velocity=0.0
- added joint Body2_Body8: type revolute, parent Body2, child Body8, origin xyz=0.314997166565409 0.2682195969029738 0 rpy=0 0 0, axis 1 0 0, limit lower=-3.14159 upper=3.14159 effort=0.0 velocity=0.0
- added joint Body3_Body12: type revolute, parent Body3, child Body12, origin xyz=0.4427521309242766 0.06353212131526666 0 rpy=0 0 0, axis 0 0 1, limit lower=-3.14159 upper=3.14159 effort=0.0 velocity=0.0
- joint Body0_Body1: axis 0 0 1 -> 1 0 0; origin xyz=0.4688980547627609 0 2.2306942307325417 rpy=0 0 0 -> xyz=0.09060715004044581 0 2.1028687496169964 rpy=0 0 0
- joint Body10_Body11: axis 1 0 0 -> 0 0 1; origin xyz=0 0.9275444579900919 -0.016931804575111214 rpy=0 0 0 -> xyz=0 -0.3393051675011771 -0.09053342464704273 rpy=0 0 0
- joint Body12_Body13: axis 0 0 1 -> 0 1 0; origin xyz=0 -0.5862782035020958 -0.1850953791795156 rpy=0 0 0 -> xyz=0 0.09174995987187068 -0.3687020729035071 rpy=0 0 0
- joint Body14_Body15: axis 1 0 0 -> 0 1 0; origin xyz=0 0.4261663683423915 -0.15404364752724883 rpy=0 0 0 -> xyz=0 -0.11039933576914382 -0.21390236107728663 rpy=0 0 0
- joint Body1_Body2: axis 0 0 1 -> 1 0 0; origin xyz=0.7179331956033698 0 0 rpy=0 0 0 -> xyz=0.7776446127363325 0 0 rpy=0 0 0
- joint Body1_Body6: origin xyz=0.3589665978016849 0.27322486278341834 0 rpy=0 0 0 -> xyz=0.3888223063681662 -0.3031000716891105 0 rpy=0 0 0
- joint Body2_Body10: axis 1 0 0 -> 0 0 1; origin xyz=0.07936923109015742 0.4724958881142447 0 rpy=0 0 0 -> xyz=0.314997166565409 -0.2682195969029738 0 rpy=0 0 0
- joint Body2_Body3: origin xyz=0.15873846218031484 0 0 rpy=0 0 0 -> xyz=0.629994333130818 0 0 rpy=0 0 0
- joint Body3_Body14: origin xyz=0.09505577408685073 0.35577648065571255 0 rpy=0 0 0 -> xyz=0.4427521309242766 -0.06353212131526666 0 rpy=0 0 0
- joint Body4_Body5: origin xyz=0.11299601147428873 0 0 rpy=0 0 0 -> xyz=0 0.34961574996824235 -0.32388025002580006 rpy=0 0 0
- joint Body6_Body7: axis 0 0 1 -> 1 0 0; origin xyz=0 0.224182805599199 -0.013406651814257077 rpy=0 0 0 -> xyz=0 -0.6285472885228587 -0.09688652419759514 rpy=0 0 0
- joint Body8_Body9: axis 0 1 0 -> 1 0 0; origin xyz=0 -0.34580592637214963 -0.04297384199435862 rpy=0 0 0 -> xyz=0 0.7678398653959259 -0.43690103163326915 rpy=0 0 0

Commit message: changed some numbers

File: body.urdf (robot description, URDF)
Before this commit: robot robot, 16 links, 15 joints
Links:
- removed link Body11
- removed link Body12
- removed link Body13
- removed link Body14
- removed link Body15
- link Body0: geometry collision box size=0.8486272748938505 0.29260892801960603 0.3098288141274208; visual box size=0.8486272748938505 0.29260892801960603 0.3098288141274208
- link Body1: geometry collision box size=0.2471748364998873 0.4500162446275928 0.6206683416137189; visual box size=0.2471748364998873 0.4500162446275928 0.6206683416137189
- link Body10: geometry collision box size=0.04422183722090096 0.10773003120856305 0.07746459858776601; visual box size=0.04422183722090096 0.10773003120856305 0.07746459858776601
- link Body2: geometry collision box size=0.1507437846696044 0.6434495778982792 0.21752206138388902; visual box size=0.1507437846696044 0.6434495778982792 0.21752206138388902
- link Body3: geometry collision box size=0.10873547612551564 0.33556366264283616 0.24033027007573135; visual box size=0.10873547612551564 0.33556366264283616 0.24033027007573135
- link Body4: geometry collision box size=0.007485651829636955 0.4168989740594981 0.06752100262644664; visual box size=0.007485651829636955 0.4168989740594981 0.06752100262644664
- link Body5: geometry collision box size=0.21882199511566672 0.6560023136086289 0.127790779509694; visual box size=0.21882199511566672 0.6560023136086289 0.127790779509694
- link Body6: geometry collision box size=0.0694339405755443 0.33715769915940713 0.07203491344749074; visual box size=0.0694339405755443 0.33715769915940713 0.07203491344749074
- link Body7: geometry collision box size=0.052323415916603035 0.30999460787566213 0.41697037932267667; visual box size=0.052323415916603035 0.30999460787566213 0.41697037932267667
- link Body8: geometry collision box size=0.030353207980681703 0.13080270924513063 0.555365928703957; visual box size=0.030353207980681703 0.13080270924513063 0.555365928703957
- link Body9: geometry collision box size=0.13908777601007513 0.4171327453046249 0.09775968094561957; visual box size=0.13908777601007513 0.4171327453046249 0.09775968094561957
Joints:
- removed joint Body10_Body11
- removed joint Body12_Body13
- removed joint Body14_Body15
- removed joint Body1_Body4
- removed joint Body1_Body6
- removed joint Body2_Body10
- removed joint Body2_Body3
- removed joint Body2_Body8
- removed joint Body3_Body12
- removed joint Body3_Body14
- removed joint Body4_Body5
- removed joint Body6_Body7
- removed joint Body8_Body9
- added joint Body1_Body3: type revolute, parent Body1, child Body3, origin xyz=0.12358741824994365 0.2250081223137964 0 rpy=0 0 0, axis 0 0 1, limit lower=-3.14159 upper=3.14159 effort=0.0 velocity=0.0
- added joint Body1_Body5: type revolute, parent Body1, child Body5, origin xyz=0.12358741824994365 -0.2250081223137964 0 rpy=0 0 0, axis 0 0 1, limit lower=-3.14159 upper=3.14159 effort=0.0 velocity=0.0
- added joint Body2_Body7: type revolute, parent Body2, child Body7, origin xyz=0.0753718923348022 0.3217247889491396 0 rpy=0 0 0, axis 0 1 0, limit lower=-3.14159 upper=3.14159 effort=0.0 velocity=0.0
- added joint Body2_Body9: type revolute, parent Body2, child Body9, origin xyz=0.0753718923348022 -0.3217247889491396 0 rpy=0 0 0, axis 0 1 0, limit lower=-3.14159 upper=3.14159 effort=0.0 velocity=0.0
- added joint Body3_Body4: type revolute, parent Body3, child Body4, origin xyz=0 0.33556366264283616 -0.12016513503786568 rpy=0 0 0, axis 1 0 0, limit lower=-3.14159 upper=3.14159 effort=0.0 velocity=0.0
- added joint Body5_Body6: type revolute, parent Body5, child Body6, origin xyz=0 -0.6560023136086289 -0.063895389754847 rpy=0 0 0, axis 0 1 0, limit lower=-3.14159 upper=3.14159 effort=0.0 velocity=0.0
- added joint Body7_Body8: type revolute, parent Body7, child Body8, origin xyz=0 0.30999460787566213 -0.20848518966133833 rpy=0 0 0, axis 0 1 0, limit lower=-3.14159 upper=3.14159 effort=0.0 velocity=0.0
- added joint Body9_Body10: type revolute, parent Body9, child Body10, origin xyz=0 -0.4171327453046249 -0.048879840472809785 rpy=0 0 0, axis 0 1 0, limit lower=-3.14159 upper=3.14159 effort=0.0 velocity=0.0
- joint Body0_Body1: origin xyz=0.09060715004044581 0 2.1028687496169964 rpy=0 0 0 -> xyz=0.42431363744692524 0 2.1549144070637105 rpy=0 0 0
- joint Body1_Body2: origin xyz=0.7776446127363325 0 0 rpy=0 0 0 -> xyz=0.2471748364998873 0 0 rpy=0 0 0

Commit message: classified everything - ready to evolve

File: body.urdf (robot description, URDF)
Before this commit: robot robot, 11 links, 10 joints
Links:
- removed link Body10
- removed link Body4
- removed link Body5
- removed link Body6
- removed link Body7
- removed link Body8
- removed link Body9
- link Body0: geometry collision box size=0.3750470351867533 0.9719076236832661 0.7162129881550383; visual box size=0.3750470351867533 0.9719076236832661 0.7162129881550383
- link Body1: geometry collision box size=0.9260028885502419 0.8108251223398693 0.5170944615239493; visual box size=0.9260028885502419 0.8108251223398693 0.5170944615239493
- link Body2: geometry collision box size=0.9192345108463461 0.17979447510176294 0.3578810374578487; visual box size=0.9192345108463461 0.17979447510176294 0.3578810374578487
- link Body3: geometry collision box size=0.11757900205900915 0.04304870560957919 0.2616971037063217; visual box size=0.11757900205900915 0.04304870560957919 0.2616971037063217
Joints:
- removed joint Body1_Body3
- removed joint Body1_Body5
- removed joint Body2_Body7
- removed joint Body2_Body9
- removed joint Body3_Body4
- removed joint Body5_Body6
- removed joint Body7_Body8
- removed joint Body9_Body10
- added joint Body2_Body3: type revolute, parent Body2, child Body3, origin xyz=0 0.17979447510176294 -0.17894051872892436 rpy=0 0 0, axis 1 0 0, limit lower=-3.14159 upper=3.14159 effort=0.0 velocity=0.0
- joint Body0_Body1: axis 1 0 0 -> 0 0 1; origin xyz=0.42431363744692524 0 2.1549144070637105 rpy=0 0 0 -> xyz=0.18752351759337665 0 2.358106494077519 rpy=0 0 0
- joint Body1_Body2: origin xyz=0.2471748364998873 0 0 rpy=0 0 0 -> xyz=0.46300144427512097 0.4054125611699346 0 rpy=0 0 0
